File: Sch/Sch.sch (EAGLE design)
At the start: 48 parts, among them IC1 MEGA8-P, IC2 TLP2630, IC3 YMZ294, IC4 YMZ294, IC5 YMZ294, IC6 74HC595, IC7 YM2413, IC8 TCXO_8MHz, IC9 NJM4558, Q1 16MHz, Q2 3.579545MHz

Commit message: Whole Changes
Parts:
- removed Q2: 3.579545MHz, crystal:CRYSTALHC49S
- removed SV5: OUTPUT, con-lstb:MA03-1
- added C16, C17, C18, C19, C20, C21: 0.1u, rcl:C-EU025-030X050
- added C23: 470u, rcl:CPOL-EUE2.5-5
- added D2, D3: 1N4148, diode:1N4148DO35-7
- added IC10: MCP2221A, ic-package:DIL14S
- added IC11: DIP-SW, ic-package:DIL8S
- added LED1: POWER, led:LED3MM
- added LED2: MIDI_IN, led:LED3MM
- added LED3: RX, led:LED3MM
- added LED4: TX, led:LED3MM
- added LED5: USBEN, led:LED3MM
- added QG1: 3.579545MHz, crystal:XO-8
- added QG2: 8MHz, crystal:XO-14
- added R17, R19: 1.2k, rcl:R-EU_0207/2V
- added R18, R20, R21, R22, R23, R28, R29: 10k, rcl:R-EU_0207/2V
- added R24, R25, R26, R27, R30: 680, rcl:R-EU_0207/2V
- added SV6: ICSP, con-lstb:MA03-2
- added SV7: USB, con-lstb:MA05-1
- added T1: 2SA1015, transistor:-PNP-TO92
- added T2: 2SD468, transistor:-NPN-TO92
- added VR1, VR2, VR3: TSR-065, akizuki:TSR-065
- C1, C2: value 0.1uF -> 22pF
- C10: value 0.1uF -> 10u; device rcl:C-EU050-025X075 -> rcl:CPOL-EUE2.5-5
- C11, C12: value 10uF -> 10u; device rcl:CPOL-EUE2.5-7 -> rcl:CPOL-EUE2.5-5
- C13, C15: value 10uF -> 0.1u; device rcl:CPOL-EUE2.5-7 -> rcl:C-EU025-030X050
- C14: value 10uF -> 100u; device rcl:CPOL-EUE2.5-7 -> rcl:CPOL-EUE2.5-5
- C3: value 22pF -> 0.1u; device rcl:C-EU050-025X075 -> rcl:C-EU025-030X050
- C4: value 22pF -> 0.015u
- C5: value 0.1uF -> 0.015u
- C6, C9: value 100uF -> 10u; device rcl:CPOL-EUE2.5-7 -> rcl:CPOL-EUE2.5-5
- C7: value (none) -> 47u; device rcl:C-EU050-025X075 -> rcl:CPOL-EUE2.5-5
- C8: value (none) -> 10u; device rcl:C-EU050-025X075 -> rcl:CPOL-EUE2.5-5
- D1: value 1N4148DO35-10 -> 1N4148; device diode:1N4148DO35-10 -> diode:1N4148DO35-7
- IC2: value TLP2630 -> 74HC595N; device ic-package:DIL8 -> 74xx-eu:74HC595N
- IC6: value 74HC595 -> YM2413; device ic-package:DIL16S -> ic-package:DIL18S
- IC7: value YM2413 -> TLP2630; device ic-package:DIL18S -> ic-package:DIL8S
- IC8: value TCXO_8MHz -> NJM2114; device ic-package:DIL14 -> ic-package:DIL8S
- IC9: value NJM4558 -> SSM2019; device ic-package:DIL8 -> ic-package:DIL8S
- R1, R11, R12, R13, R14, R15, R16, R2, R8: device rcl:R-EU_0207/10 -> rcl:R-EU_0207/2V
- R10, R4, R6: value 10k -> 2.2k; device rcl:R-EU_0207/10 -> rcl:R-EU_0207/2V
- R3: value 1k -> 10k; device rcl:R-EU_0207/10 -> rcl:R-EU_0207/2V
- R5: value 10k -> 4.7k; device rcl:R-EU_0207/10 -> rcl:R-EU_0207/2V
- R7: value 1.2k -> 4.7k; device rcl:R-EU_0207/10 -> rcl:R-EU_0207/2V
- R9: value 1.2k -> 10k; device rcl:R-EU_0207/10 -> rcl:R-EU_0207/2V
- SV1: value ICSP -> MIDI_IN; device con-lstb:MA03-2 -> con-lstb:MA05-1
- SV2: value MIDI_IN -> VR; device con-lstb:MA05-1 -> con-lstb:MA03-1
- SV3: value POWER -> OUT; device con-lstb:MA04-1 -> con-lstb:MA03-1
- SV4: value VR -> POWER
Connections:
- removed net +5V: C2.1, C6.+, IC1.AVCC, IC1.VCC@1, IC3.4, IC4.4, IC5.4, IC6.10, IC6.16, IC7.16, IC8.1, IC8.2, IC8.3, IC9.8, R1.2, R5.2, SV1.2, SV3.1, SV3.4
- removed net N$28: IC3.7, IC4.7, IC5.7, IC8.12, IC8.13, IC8.14
- removed net N$34: IC1.PB0(ICP), IC6.14
- removed net N$35: IC1.PB1(OC1A), IC6.12
- removed net N$36: IC1.PB2(SS/OC1B), IC6.11
- removed net N$37: C10.1, IC9.3, R5.1, R6.2
- removed net N$38: C9.-, R4.2, SV5.1, SV5.3
- removed net N$39: IC3.5, R7.2, R8.2
- removed net N$40: C11.-, R8.1
- removed net N$41: IC4.5, R10.2, R9.2
- removed net N$42: C12.-, R10.1
- removed net N$43: IC5.5, R11.2, R12.2
- removed net N$44: C13.-, R12.1
- removed net N$45: R13.2, R14.2
- removed net N$46: C14.-, R14.1
- removed net N$47: IC7.14, R15.2, R16.2
- removed net N$48: C15.-, R16.1
- removed net N$49: IC1.PD0(RXD), IC2.7, R3.1
- new net A0: IC1.PD6(AIN0), IC3.3, IC4.3, IC5.3, IC6.10
- new net CONFIG1: IC1.PB0(ICP), IC11.3, R29.2
- new net CONFIG2: IC1.PB1(OC1A), IC11.4, R28.2
- new net D+: IC10.13, SV7.3
- new net D-: IC10.12, SV7.2
- new net DATA0: IC2A.QA, IC3.18, IC4.18, IC5.18, IC6.17
- new net DATA1: IC2A.QB, IC3.17, IC4.17, IC5.17, IC6.18
- new net DATA2: IC2A.QC, IC3.16, IC4.16, IC5.16, IC6.2
- new net DATA3: IC2A.QD, IC3.15, IC4.15, IC5.15, IC6.3
- new net DATA4: IC2A.QE, IC3.14, IC4.14, IC5.14, IC6.4
- new net DATA5: IC2A.QF, IC3.13, IC4.13, IC5.13, IC6.5
- new net DATA6: IC2A.QG, IC3.12, IC4.12, IC5.12, IC6.6
- new net DATA7: IC2A.QH, IC3.11, IC4.11, IC5.11, IC6.7
- new net FM_CS: IC1.PD5(T1), IC6.12
- new net FM_MO: IC6.14, R6.2, R7.2
- new net FM_RO: IC6.15, R4.2, R5.2
- new net FM_WE: IC1.PD4(XCK/T0), IC6.11
- new net GP0: IC10.2, LED3.C
- new net GP1: IC10.3, LED4.C
- new net GP2: IC10.7, LED5.C
- new net IC: D2.C, IC1.PD7(AIN1), IC3.9, IC4.9, IC5.9, IC6.13
- new net MIDI_IN: IC11.8, IC7.7, LED2.C, R3.1
- new net MISO: IC1.PB4(MISO), SV6.1
- new net MOSI: IC1.PB3(MOSI/OC2), IC2A.SER, SV6.4
- new net N$14: C7.+, D3.C, T1.E
- new net NC: SV7.4
- new net PSG1_CS: IC1.PC1(ADC1), IC3.2
- new net PSG1_OUT: IC3.5, R19.2, R20.2
- new net PSG1_WR: IC1.PC0(ADC0), IC3.1
- new net PSG2_CS: IC1.PC3(ADC3), IC4.2
- new net PSG2_OUT: IC4.5, R17.2, R18.2
- new net PSG2_WR: IC1.PC2(ADC2), IC4.1
- new net PSG3_CS: IC1.PC5(ADC5/SCL), IC5.2
- new net PSG3_OUT: IC5.5, R15.2, R16.2
- new net PSG3_WR: IC1.PC4(ADC4/SDA), IC5.1
- new net RCK: IC1.PB2(SS/OC1B), IC2A.RCK
- new net RST: IC1.PC6(/RESET), R1.1, SV6.5
- new net RX: IC1.PD0(RXD), IC11.1, IC11.2
- new net SCK: IC1.PB5(SCK), IC2A.SCK, SV6.3
- new net TX: IC1.PD1(TXD), IC10.5
- new net USB_RX: IC10.6, IC11.7
- new net VBAS: IC10.1, SV7.1
- new net VBIAS: C13.1, IC8.3, R21.1, R22.2
- new net VCC: C15.1, C16.1, C17.1, C18.1, C19.1, C20.1, C21.1, C23.+, C3.1, D3.A, IC1.AVCC, IC1.VCC@1, IC11.5, IC11.6, IC2A.SCL, IC3.4, IC4.4, IC5.4, IC6.16, IC7.8, IC8.8, IC9.7, QG1.VCC, QG2.VCC, R1.2, R21.2, R24.2, R25.2, R26.2, R27.2, R3.2, R30.2, R9.2, SV4.2, SV6.2
- net GND: now also C1.2, C13.2, C15.2, C16.2, C17.2, C18.2, C19.2, C20.2, C21.2, C23.-, C3.2, C4.2, C5.2, C7.-, IC1.AREF, IC10.14, IC2A.G, IC6.1, IC7.5, IC8.4, IC9.2, LED1.C, QG1.GND, QG2.GND, R17.1, R19.1, R22.1, R23.1, R28.1, R29.1, SV4.1, SV4.3, SV6.6, SV7.5, T2.C; no longer C1.1, C10.2, C3.1, C4.1, C7.1, C8.1, IC6.13, IC6.8, IC7.1, IC8.10, IC8.8, IC8.9, R7.1, R9.1, SV1.6, SV3.3, SV5.2
- net N$1: now also R2.1, SV1.4; no longer IC1.PC6(/RESET), R1.1, SV1.5
- net N$10: now also C10.+, C11.+, C12.+, C8.+, C9.+, IC8.2, VR3.A, VR3.S; no longer R2.1, SV2.5
- net N$11: now also C5.1, R7.1, VR2.A, VR2.S; no longer D1.C, IC2.1, R2.2
- net N$12: now also LED3.A, R24.1; no longer C5.1, IC2.8, R3.2
- net N$13: now also R8.2, R9.1, T1.B; no longer C5.2, IC2.5
- net N$15: now also R10.1, T1.C; no longer IC1.PD3(INT1), IC3.1, IC3.2
- net N$16: now also R10.2, T2.B; no longer IC3.11, IC4.11, IC5.11, IC6.7, IC7.7
- net N$17: now also C14.-, IC9.3, R23.2, T2.E; no longer IC3.12, IC4.12, IC5.12, IC6.6, IC7.6
- net N$18: now also R11.2, R12.2, VR2.E; no longer IC3.13, IC4.13, IC5.13, IC6.5, IC7.5
- net N$19: now also C8.-, R12.1; no longer IC3.14, IC4.14, IC5.14, IC6.4, IC7.4
- net N$2: now also D1.A, IC7.2, SV1.5; no longer IC1.PB3(MOSI/OC2), SV1.4
- net N$20: now also R13.2, R14.2, VR1.E; no longer IC3.15, IC4.15, IC5.15, IC6.3, IC7.3
- net N$21: now also C9.-, R14.1; no longer IC3.16, IC4.16, IC5.16, IC6.2, IC7.2
- net N$22: now also LED4.A, R25.1; no longer IC3.17, IC4.17, IC5.17, IC6.1, IC7.18
- net N$23: now also C10.-, R16.1; no longer IC1.PD4(XCK/T0), IC4.1, IC4.2
- net N$24: now also LED5.A, R30.1; no longer IC1.PD5(T1), IC5.1, IC5.2
- net N$25: now also C11.-, R18.1; no longer IC1.PD6(AIN0), IC3.3, IC4.3, IC5.3, IC7.10
- net N$26: now also LED1.A, R26.1; no longer C11.+, C12.+, C13.+, C14.+, C15.+, IC9.2, SV4.2, SV4.3
- net N$27: now also C12.-, R20.1; no longer IC1.PD2(INT0), IC7.11, IC7.12
- net N$29: now also C14.+, IC8.1, VR3.E; no longer IC8.5, IC8.6, IC8.7
- net N$3: now also C1.1, IC1.PB6(XTAL1/TOSC1), Q1.2; no longer IC1.PB4(MISO), SV1.1
- net N$30: now also IC9.1, SV2.1, SV2.2; no longer IC1.PD7(AIN1), IC3.9, IC4.9, IC5.9, IC7.13
- net N$31: now also IC9.8, SV2.3; no longer C9.+, IC9.1, SV4.1
- net N$32: now also LED2.A, R27.1; no longer C7.2, IC7.8, Q2.2
- net N$33: now also IC9.6, SV3.1, SV3.3; no longer C8.2, IC7.9, Q2.1
- net N$4: now also C2.1, IC1.PB7(XTAL2/TOSC2), Q1.1; no longer C1.2, IC1.AREF
- net N$5: now also D1.C, IC7.1, R2.2; no longer C3.2, IC1.PB6(XTAL1/TOSC1), Q1.2
- net N$6: now also IC3.7, IC4.7, IC5.7, QG2.OUT; no longer C4.2, IC1.PB7(XTAL2/TOSC2), Q1.1
- net N$7: now also C6.+, D2.A, R8.1; no longer IC1.PB5(SCK), SV1.3
- net N$8: now also C4.1, R5.1, VR1.A, VR1.S; no longer IC3.18, IC4.18, IC5.18, IC6.15, IC7.17
- net N$9: now also IC6.8, QG1.OUT; no longer D1.A, IC2.2, SV2.4
Other:
- note added: "0.015u capacitors use film capacitor"
- note added: "HARDWARE MIDI TONE GENERATOR -HiT0M1"
- note added: "Vcc=5v GND=0v"
- note added: "Ver2.40"
- moved on the sheet: C1, C11, C12, C14, C2, C3, C4, C5, C6, C9, D1, IC1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

Commit message: Update Readme.md
Parts:
- removed IC2: 74HC595N, 74xx-eu:74HC595N
- added SV5: LCD, con-lstb:MA07-2
- added VR4: TSR-065, akizuki:TSR-065
- IC1: value MEGA8-P -> MEGA32-P; device atmel:MEGA8-P -> atmel:MEGA32-P
Connections:
- removed net N$3: C1.1, IC1.PB6(XTAL1/TOSC1), Q1.2
- removed net RCK: IC1.PB2(SS/OC1B), IC2A.RCK
- new net DB4: IC1.(OC1B)PD4, SV5.11
- new net DB5: IC1.(OC1A)PD5, SV5.12
- new net DB6: IC1.(ICP)PD6, SV5.13
- new net DB7: IC1.(OC2)PD7, SV5.14
- new net E: IC1.(AIN0/INT2)PB2, SV5.6
- new net N$28: C1.1, IC1.XTAL2, Q1.2
- new net N$38: SV5.8
- new net N$39: SV5.10
- new net N$44: SV5.7
- new net N$45: SV5.9
- new net R/W: IC1.(T0/XCK)PB0, SV5.5
- new net RS: IC1.(T1)PB1, SV5.4
- new net VO: SV5.3, VR4.A, VR4.S
- net A0: now also IC1.(SS)PB4; no longer IC1.PD6(AIN0)
- net CONFIG1: now also IC1.(INT0)PD2; no longer IC1.PB0(ICP)
- net CONFIG2: now also IC1.(INT1)PD3; no longer IC1.PB1(OC1A)
- net DATA0: now also IC1.(ADC0)PA0; no longer IC2A.QA
- net DATA1: now also IC1.(ADC1)PA1; no longer IC2A.QB
- net DATA2: now also IC1.(ADC2)PA2; no longer IC2A.QC
- net DATA3: now also IC1.(ADC3)PA3; no longer IC2A.QD
- net DATA4: now also IC1.(ADC4)PA4; no longer IC2A.QE
- net DATA5: now also IC1.(ADC5)PA5; no longer IC2A.QF
- net DATA6: now also IC1.(ADC6)PA6; no longer IC2A.QG
- net DATA7: now also IC1.(ADC7)PA7; no longer IC2A.QH
- net FM_CS: now also IC1.(TOSC2)PC7; no longer IC1.PD5(T1)
- net FM_WE: now also IC1.(TOSC1)PC6; no longer IC1.PD4(XCK/T0)
- net GND: now also SV5.2, VR4.E; no longer IC2A.G
- net IC: now also IC1.(AIN1/OC0)PB3; no longer IC1.PD7(AIN1)
- net MISO: now also IC1.(MISO)PB6; no longer IC1.PB4(MISO)
- net MOSI: now also IC1.(MOSI)PB5; no longer IC1.PB3(MOSI/OC2), IC2A.SER
- net N$4: now also IC1.XTAL1; no longer IC1.PB7(XTAL2/TOSC2)
- net PSG1_CS: now also IC1.(SDA)PC1; no longer IC1.PC1(ADC1)
- net PSG1_WR: now also IC1.(SCL)PC0; no longer IC1.PC0(ADC0)
- net PSG2_CS: now also IC1.(TMS)PC3; no longer IC1.PC3(ADC3)
- net PSG2_WR: now also IC1.(TCK)PC2; no longer IC1.PC2(ADC2)
- net PSG3_CS: now also IC1.(TDI)PC5; no longer IC1.PC5(ADC5/SCL)
- net PSG3_WR: now also IC1.(TDO)PC4; no longer IC1.PC4(ADC4/SDA)
- net RST: now also IC1.RESET; no longer IC1.PC6(/RESET)
- net RX: now also IC1.(RXD)PD0; no longer IC1.PD0(RXD)
- net SCK: now also IC1.(SCK)PB7; no longer IC1.PB5(SCK), IC2A.SCK
- net TX: now also IC1.(TXD)PD1; no longer IC1.PD1(TXD)
- net VCC: now also IC1.VCC, SV5.1; no longer IC1.VCC@1, IC2A.SCL
Other:
- moved on the sheet: C1, C2, Q1, R1
