File: Schematic/Sch.brd (EAGLE design)
At the start: 100 x 100 mm, 86 parts, among them IC1 MEGA32-P, IC10 MCP2221A, IC11 DIP-SW, IC3 YMZ294, IC4 YMZ294, IC5 YMZ294, IC6 YM2413, IC7 TLP2630, IC8 NJM2114, IC9 SSM2019, Q1 16MHz, T1 2SA1015, T2 2SD468

Commit message: Whole Changes
Parts:
- removed D2, D3: 1N4148, diode:DO35-7
- removed IC10: MCP2221A, ic-package:SOCKET-14
- removed IC11: DIP-SW, ic-package:SOCKET-08
- removed QG2: 8MHz, crystal:DIL14S
- removed R21, R22, R23, R28, R29: 10k, rcl:0207/2V
- removed R24, R25, R26, R27, R30: 680, rcl:0207/2V
- removed SV6: ICSP, con-lstb:MA03-2
- removed SV7: USB, con-lstb:MA05-1
- removed T1: 2SA1015, transistor:TO92
- removed T2: 2SD468, transistor:TO92
- removed VR1, VR4: TSR-065, akizuki:TSR-065
- added C22: 0.1u, rcl:C025-025X050
- added IC2: 74HC139N, 74xx-eu:DIL16
- added LED6: WITH_R, led:LED3MM
- added Q2: 3.579545MHz, crystal:HC49/S
- C1, C2: value 22pF -> 22p; device rcl:C050-025X075 -> rcl:C025-025X050
- C10, C11, C12, C23, C8, C9: device rcl:E2,5-5 -> rcl:E2,5-6
- C13: value 0.1u -> 0.015u; device rcl:C025-030X050 -> rcl:C050-025X075
- C14: value 100u -> 0.015u; device rcl:E2,5-5 -> rcl:C050-025X075
- C15, C16, C17, C18, C19, C20, C21, C3: device rcl:C025-030X050 -> rcl:C025-025X050
- C4, C5: value 0.015u -> 22p; device rcl:C050-025X075 -> rcl:C025-025X050
- C6: value 10u -> 100u; device rcl:E2,5-5 -> rcl:E2,5-6
- C7: value 47u -> 0.1u; device rcl:E2,5-5 -> rcl:C025-025X050
- IC1: value MEGA32-P -> MEGA328P; device atmel:DIL40 -> atmel:DIL28-3
- IC3: value YMZ294 -> 74HC595N; device ic-package:SOCKET-18 -> 74xx-eu:DIL16
- IC6: value YM2413 -> YMZ294
- IC7: value TLP2630 -> YM2413; device ic-package:SOCKET-08 -> ic-package:SOCKET-18
- IC8: value NJM2114 -> TLP2630
- IC9: value SSM2019 -> NJM2114
- LED1: value POWER -> WITH_R
- LED2: value MIDI_IN -> WITH_R
- LED3: value RX -> WITH_R
- LED4: value TX -> WITH_R
- LED5: value USBEN -> WITH_R
- QG1: value 3.579545MHz -> 8MHz; device crystal:DIL08S -> crystal:DIL14S
- R1, R2: device rcl:0207/2V -> rcl:0207/10
- R10: value 2.2k -> 10k
- R17: value 1.2k -> 4.7k
- R18: value 10k -> 4.7k
- R19: value 1.2k -> 2.2k
- R20: value 10k -> 2.2k
- R3: value 10k -> 1k; device rcl:0207/2V -> rcl:0207/10
- R4, R6: value 2.2k -> 10k; device rcl:0207/2V -> rcl:0207/10
- R5: value 4.7k -> 10k; device rcl:0207/2V -> rcl:0207/10
- R7: value 4.7k -> 1.2k
- R9: value 10k -> 1.2k
- SV1: value MIDI_IN -> ICSP; device con-lstb:MA05-1 -> con-lstb:MA03-2
- SV2: value VR -> MIDI_IN; device con-lstb:MA03-1 -> con-lstb:MA05-1
- SV3: value OUT -> POWER
- SV4: value POWER -> OUT
- SV5: value LCD -> VOL; device con-lstb:MA07-2 -> con-lstb:MA03-1
- VR2, VR3: value TSR-065 -> VR_3362P; device akizuki:TSR-065 -> Akizuki:VR_3362P
- moved LED1 118.4 mm to (77.5, 3.81)
- moved SV5 111.3 mm to (6.35, 3.81)
- moved LED2 107.0 mm to (67.3, 3.81)
- moved C23 103.4 mm to (15.2, 95.2), turned to 0 degrees
- moved LED3 98.4 mm to (57.1, 3.81)
- moved C6 94.2 mm to (88.9, 10.2)
- moved LED4 93.6 mm to (47.0, 3.81)
- moved LED5 93.0 mm to (36.8, 3.81)
- moved SV3 88.9 mm to (6.35, 95.2)
- moved C2 88.6 mm to (14.0, 74.9), turned to 90 degrees
- moved C1 86.6 mm to (14.0, 85.1), turned to 270 degrees
- moved Q1 86.4 mm to (7.62, 80.0)
- moved R4 80.2 mm to (95.2, 12.7)
- moved SV1 77.5 mm to (64.8, 80.0), turned to 90 degrees
- moved VR3 74.9 mm to (55.9, 11.4)
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Connections:
- removed net CONFIG1: IC1.16, IC11.3, R29.2
- removed net CONFIG2: IC1.17, IC11.4, R28.2
- removed net D+: IC10.13, SV7.3
- removed net D-: IC10.12, SV7.2
- removed net DB4: IC1.18, SV5.11
- removed net DB5: IC1.19, SV5.12
- removed net DB6: IC1.20, SV5.13
- removed net DB7: IC1.21, SV5.14
- removed net E: IC1.3, SV5.6
- removed net FM_MO: IC6.14, R6.2, R7.2
- removed net FM_RO: IC6.15, R4.2, R5.2
- removed net FM_WE: IC1.28, IC6.11
- removed net GP0: IC10.2, LED3.K
- removed net GP1: IC10.3, LED4.K
- removed net GP2: IC10.7, LED5.K
- removed net N$12: LED3.A, R24.1
- removed net N$16: R10.2, T2.2
- removed net N$25: C11.-, R18.1
- removed net N$26: LED1.A, R26.1
- removed net N$27: C12.-, R20.1
- removed net N$28: C1.1, IC1.12, Q1.2
- removed net N$29: C14.+, IC8.1, VR3.3
- removed net N$30: IC9.1, SV2.1, SV2.2
- removed net N$31: IC9.8, SV2.3
- removed net N$32: LED2.A, R27.1
- removed net N$33: IC9.6, SV3.1, SV3.3
- removed net N$38: SV5.8
- removed net N$39: SV5.10
- removed net N$44: SV5.7
- removed net N$45: SV5.9
- removed net N$6: IC3.7, IC4.7, IC5.7, QG2.8
- removed net N$9: IC6.8, QG1.5
- removed net NC: SV7.4
- removed net R/W: IC1.1, SV5.5
- removed net RS: IC1.2, SV5.4
- removed net RX: IC1.14, IC11.1, IC11.2
- removed net TX: IC1.15, IC10.5
- removed net USB_RX: IC10.6, IC11.7
- removed net VBAS: IC10.1, SV7.1
- removed net VO: SV5.3, VR4.1, VR4.2
- new net CS_A: IC1.23, IC2.2
- new net CS_B: IC1.24, IC2.3
- new net CS_E: IC1.14, IC2.1
- new net FMM_LED: IC1.13, LED5.A
- new net FMM_OUT: IC7.14, R17.2, R19.1
- new net FMR_LED: IC1.12, LED4.A
- new net FMR_OUT: IC7.15, R18.2, R20.1
- new net FM_CLKIN: C4.2, IC7.8, Q2.2
- new net FM_CLKOUT: C5.2, IC7.9, Q2.1
- new net FM_WR: IC2.9, IC7.11
- new net N$3: D1.C, IC8.1, R2.2
- new net OUT: C6.-, R4.2
- new net PSG1_LED: IC1.5, LED1.A
- new net PSG2_LED: IC1.6, LED2.A
- new net PSG3_LED: IC1.11, LED3.A
- new net PSG_CLK: IC4.7, IC5.7, IC6.7, QG1.8
- new net RCK: IC1.16, IC3.12
- new net WR_A: IC1.25, IC2.14
- new net WR_B: IC1.26, IC2.13
- new net WR_E: IC1.15, IC2.15
- net A0: now also IC1.28, IC6.3, IC7.10; no longer IC1.5, IC3.3, IC6.10
- net DATA0: now also IC3.15, IC6.18, IC7.17; no longer IC1.40, IC3.18, IC6.17
- net DATA1: now also IC3.1, IC6.17, IC7.18; no longer IC1.39, IC3.17, IC6.18
- net DATA2: now also IC3.2, IC6.16, IC7.2; no longer IC1.38, IC3.16, IC6.2
- net DATA3: now also IC3.3, IC6.15, IC7.3; no longer IC1.37, IC3.15, IC6.3
- net DATA4: now also IC3.4, IC6.14, IC7.4; no longer IC1.36, IC3.14, IC6.4
- net DATA5: now also IC3.5, IC6.13, IC7.5; no longer IC1.35, IC3.13, IC6.5
- net DATA6: now also IC3.6, IC6.12, IC7.6; no longer IC1.34, IC3.12, IC6.6
- net DATA7: now also IC3.7, IC6.11, IC7.7; no longer IC1.33, IC3.11, IC6.7
- net FM_CS: now also IC2.7, IC7.12; no longer IC1.29, IC6.12
- net GND: now also C1.1, C14.2, C2.1, C22.2, C4.1, C5.1, C7.2, IC1.21, IC1.22, IC1.8, IC2.8, IC3.13, IC6.6, IC6.8, IC7.1, LED2.K, LED3.K, LED4.K, LED5.K, QG1.7, R19.2, R20.2, R7.1, R9.1, SV1.6, SV3.1, SV3.3; no longer C1.2, C2.2, C3.2, C4.2, C5.2, C6.-, C7.-, IC1.11, IC1.31, IC1.32, IC10.14, IC3.6, IC6.1, IC7.5, IC8.4, IC9.2, QG1.4, QG2.7, R17.1, R19.1, R22.1, R23.1, R28.1, R29.1, SV3.2, SV4.1, SV4.3, SV5.2, SV6.6, SV7.5, T2.3, VR4.3
- net IC: now also IC1.27, IC6.9, IC7.13; no longer D2.C, IC1.4, IC3.9, IC6.13
- net MIDI_IN: now also IC1.2, IC8.7, LED6.K; no longer IC11.8, IC7.7, LED2.K
- net MISO: now also IC1.18, SV1.1; no longer IC1.7, SV6.1
- net MOSI: now also IC1.17, IC3.14, SV1.4; no longer IC1.6, SV6.4
- net N$1: now also C1.2, IC1.9, Q1.2; no longer R2.1, SV1.4
- net N$10: now also C8.-, R8.1; no longer C10.+, C11.+, C12.+, C8.+, C9.+, IC8.2, VR3.1, VR3.2
- net N$11: now also IC4.10; no longer C5.1, R7.1, VR2.1, VR2.2
- net N$13: now also IC6.10; no longer R8.2, R9.1, T1.2
- net N$14: now also C2.2, IC1.10, Q1.1; no longer C7.+, D3.C, T1.1
- net N$15: now also C9.-; no longer T1.3
- net N$17: now also C10.-, R12.1; no longer C14.-, IC9.3, R23.2, T2.1
- net N$18: now also R13.2, R14.2, VR2.1; no longer R11.2, R12.2, VR2.3
- net N$19: now also C11.-, R14.1; no longer C8.-, R12.1
- net N$2: now also R2.1, SV2.4; no longer D1.A, IC7.2, SV1.5
- net N$20: now also R15.2, R16.2, VR3.1; no longer R13.2, R14.2, VR1.3
- net N$21: now also C12.-, R16.1; no longer C9.-, R14.1
- net N$22: now also C14.1, R18.1, VR3.2, VR3.3; no longer LED4.A, R25.1
- net N$23: now also C10.+, C11.+, C12.+, C8.+, C9.+, IC9.2, SV5.1; no longer C10.-, R16.1
- net N$24: now also C13.1, R17.1, VR2.2, VR2.3; no longer LED5.A, R30.1
- net N$4: now also D1.A, IC8.2, SV2.5; no longer C2.1, IC1.13, Q1.1
- net N$5: now also C3.2, IC8.5; no longer D1.C, IC7.1, R2.2
- net N$7: now also IC9.1, SV5.2, SV5.3; no longer D2.A, R8.1
- net N$8: now also IC5.10; no longer C4.1, R5.1, VR1.1, VR1.2
- net PSG1_CS: now also IC2.4, IC4.2; no longer IC1.23, IC3.2
- net PSG1_OUT: now also IC4.5, R7.2, R8.2; no longer IC3.5, R19.2, R20.2
- net PSG1_WR: now also IC2.12, IC4.1; no longer IC1.22, IC3.1
- net PSG2_CS: now also IC2.5, IC5.2; no longer IC1.25, IC4.2
- net PSG2_OUT: now also IC5.5, R10.2, R9.2; no longer IC4.5, R17.2, R18.2
- net PSG2_WR: now also IC2.11, IC5.1; no longer IC1.24, IC4.1
- net PSG3_CS: now also IC2.6, IC6.2; no longer IC1.27, IC5.2
- net PSG3_OUT: now also IC6.5, R11.2, R12.2; no longer IC5.5, R15.2, R16.2
- net PSG3_WR: now also IC2.10, IC6.1; no longer IC1.26, IC5.1
- net RST: now also IC1.1, R1.2, SV1.5; no longer IC1.9, R1.1, SV6.5
- net SCK: now also IC1.19, IC3.11, SV1.3; no longer IC1.8, SV6.3
- net VBIAS: now also C7.1, IC9.3, R5.1, R6.2; no longer C13.1, IC8.3, R21.1, R22.2
- net VCC: now also C22.1, IC1.20, IC1.7, IC2.16, IC3.10, IC3.16, IC6.4, IC7.16, IC9.8, LED6.A, QG1.14, R1.1, R5.2, SV1.2, SV3.2; no longer D3.A, IC1.10, IC1.30, IC11.5, IC11.6, IC3.4, IC6.16, IC7.8, IC9.7, QG1.8, QG2.14, R1.2, R21.2, R24.2, R25.2, R26.2, R27.2, R30.2, R9.2, SV4.2, SV5.1, SV6.2
Routing:
- net PSG1_LED: track 0.00 -> 187.5 mm, vias 0 -> 2
- net PSG3_LED: track 0.00 -> 182.4 mm
- net PSG2_LED: track 0.00 -> 156.6 mm, vias 0 -> 4
- net FMM_LED: track 0.00 -> 148.6 mm, vias 0 -> 3
- net GP2: track 136.4 -> 0.00 mm, vias 2 -> 0
- net GP1: track 127.7 -> 0.00 mm, vias 1 -> 0
- net DATA5: track 76.0 -> 198.2 mm, vias 4 -> 3
- net N$23: track 8.19 -> 128.9 mm, vias 0 -> 2
- net FM_WR: track 0.00 -> 119.3 mm, vias 0 -> 2
- net GND: track 689.9 -> 577.5 mm, vias 0 -> 6
- net PSG3_WR: track 137.2 -> 32.6 mm, vias 1 -> 0
- net DB4: track 97.9 -> 0.00 mm
- net R/W: track 91.2 -> 0.00 mm, vias 4 -> 0
- net GP0: track 88.4 -> 0.00 mm, vias 6 -> 0
- net N$7: track 47.6 -> 134.2 mm
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- removed copper zone on layer 1, net GND
- removed copper zone on layer 16, net GND
Other:
- board text added: "HiT0M1 Ver2.80"
- board text added: "Ivory Aveline Haskell"
- board text removed: "C:/Users/Ivory/Desktop/idesa.bmp"
