File: Schematic/Sch.sch (EAGLE design)
At the start: 86 parts, among them IC1 MEGA32-P, IC10 MCP2221A, IC11 DIP-SW, IC3 YMZ294, IC4 YMZ294, IC5 YMZ294, IC6 YM2413, IC7 TLP2630, IC8 NJM2114, IC9 SSM2019, Q1 16MHz, T1 2SA1015, T2 2SD468

Commit message: Whole Changes
Parts:
- removed D2, D3: 1N4148, diode:1N4148DO35-7
- removed IC10: MCP2221A, ic-package:DIL14S
- removed IC11: DIP-SW, ic-package:DIL8S
- removed QG2: 8MHz, crystal:XO-14
- removed R21, R22, R23, R28, R29: 10k, rcl:R-EU_0207/2V
- removed R24, R25, R26, R27, R30: 680, rcl:R-EU_0207/2V
- removed SV6: ICSP, con-lstb:MA03-2
- removed SV7: USB, con-lstb:MA05-1
- removed T1: 2SA1015, transistor:-PNP-TO92
- removed T2: 2SD468, transistor:-NPN-TO92
- removed VR1, VR4: TSR-065, akizuki:TSR-065
- added C22: 0.1u, rcl:C-EU025-025X050
- added IC2: 74HC139N, 74xx-eu:74HC139N
- added LED6: WITH_R, led:LED3MM
- added Q2: 3.579545MHz, crystal:CRYSTALHC49S
- C1, C2: value 22pF -> 22p; device rcl:C-EU050-025X075 -> rcl:C-EU025-025X050
- C10, C11, C12, C23, C8, C9: device rcl:CPOL-EUE2.5-5 -> rcl:CPOL-EUE2.5-6
- C13: value 0.1u -> 0.015u; device rcl:C-EU025-030X050 -> rcl:C-EU050-025X075
- C14: value 100u -> 0.015u; device rcl:CPOL-EUE2.5-5 -> rcl:C-EU050-025X075
- C15, C16, C17, C18, C19, C20, C21, C3: device rcl:C-EU025-030X050 -> rcl:C-EU025-025X050
- C4, C5: value 0.015u -> 22p; device rcl:C-EU050-025X075 -> rcl:C-EU025-025X050
- C6: value 10u -> 100u; device rcl:CPOL-EUE2.5-5 -> rcl:CPOL-EUE2.5-6
- C7: value 47u -> 0.1u; device rcl:CPOL-EUE2.5-5 -> rcl:C-EU025-025X050
- IC1: value MEGA32-P -> MEGA328P; device atmel:MEGA32-P -> atmel:MEGA8-P
- IC3: value YMZ294 -> 74HC595N; device ic-package:DIL18S -> 74xx-eu:74HC595N
- IC6: value YM2413 -> YMZ294
- IC7: value TLP2630 -> YM2413; device ic-package:DIL8S -> ic-package:DIL18S
- IC8: value NJM2114 -> TLP2630
- IC9: value SSM2019 -> NJM2114
- LED1: value POWER -> WITH_R
- LED2: value MIDI_IN -> WITH_R
- LED3: value RX -> WITH_R
- LED4: value TX -> WITH_R
- LED5: value USBEN -> WITH_R
- QG1: value 3.579545MHz -> 8MHz; device crystal:XO-8 -> crystal:XO-14
- R1, R2: device rcl:R-EU_0207/2V -> rcl:R-EU_0207/10
- R10: value 2.2k -> 10k
- R17: value 1.2k -> 4.7k
- R18: value 10k -> 4.7k
- R19: value 1.2k -> 2.2k
- R20: value 10k -> 2.2k
- R3: value 10k -> 1k; device rcl:R-EU_0207/2V -> rcl:R-EU_0207/10
- R4, R6: value 2.2k -> 10k; device rcl:R-EU_0207/2V -> rcl:R-EU_0207/10
- R5: value 4.7k -> 10k; device rcl:R-EU_0207/2V -> rcl:R-EU_0207/10
- R7: value 4.7k -> 1.2k
- R9: value 10k -> 1.2k
- SV1: value MIDI_IN -> ICSP; device con-lstb:MA05-1 -> con-lstb:MA03-2
- SV2: value VR -> MIDI_IN; device con-lstb:MA03-1 -> con-lstb:MA05-1
- SV3: value OUT -> POWER
- SV4: value POWER -> OUT
- SV5: value LCD -> VOL; device con-lstb:MA07-2 -> con-lstb:MA03-1
- VR2, VR3: value TSR-065 -> VR_3362P; device akizuki:TSR-065 -> Akizuki:P-03277_VR_3362P
Connections:
- removed net CONFIG1: IC1.(INT0)PD2, IC11.3, R29.2
- removed net CONFIG2: IC1.(INT1)PD3, IC11.4, R28.2
- removed net D+: IC10.13, SV7.3
- removed net D-: IC10.12, SV7.2
- removed net DB4: IC1.(OC1B)PD4, SV5.11
- removed net DB5: IC1.(OC1A)PD5, SV5.12
- removed net DB6: IC1.(ICP)PD6, SV5.13
- removed net DB7: IC1.(OC2)PD7, SV5.14
- removed net E: IC1.(AIN0/INT2)PB2, SV5.6
- removed net FM_MO: IC6.14, R6.2, R7.2
- removed net FM_RO: IC6.15, R4.2, R5.2
- removed net FM_WE: IC1.(TOSC1)PC6, IC6.11
- removed net GP0: IC10.2, LED3.C
- removed net GP1: IC10.3, LED4.C
- removed net GP2: IC10.7, LED5.C
- removed net N$12: LED3.A, R24.1
- removed net N$16: R10.2, T2.B
- removed net N$25: C11.-, R18.1
- removed net N$26: LED1.A, R26.1
- removed net N$27: C12.-, R20.1
- removed net N$28: C1.1, IC1.XTAL2, Q1.2
- removed net N$29: C14.+, IC8.1, VR3.E
- removed net N$30: IC9.1, SV2.1, SV2.2
- removed net N$31: IC9.8, SV2.3
- removed net N$32: LED2.A, R27.1
- removed net N$33: IC9.6, SV3.1, SV3.3
- removed net N$38: SV5.8
- removed net N$39: SV5.10
- removed net N$44: SV5.7
- removed net N$45: SV5.9
- removed net N$6: IC3.7, IC4.7, IC5.7, QG2.OUT
- removed net N$9: IC6.8, QG1.OUT
- removed net NC: SV7.4
- removed net R/W: IC1.(T0/XCK)PB0, SV5.5
- removed net RS: IC1.(T1)PB1, SV5.4
- removed net RX: IC1.(RXD)PD0, IC11.1, IC11.2
- removed net TX: IC1.(TXD)PD1, IC10.5
- removed net USB_RX: IC10.6, IC11.7
- removed net VBAS: IC10.1, SV7.1
- removed net VO: SV5.3, VR4.A, VR4.S
- new net CS_A: IC1.PC0(ADC0), IC2A.A
- new net CS_B: IC1.PC1(ADC1), IC2A.B
- new net CS_E: IC1.PB0(ICP), IC2A.G
- new net FMM_LED: IC1.PD7(AIN1), LED5.A
- new net FMM_OUT: IC7.14, R17.2, R19.1
- new net FMR_LED: IC1.PD6(AIN0), LED4.A
- new net FMR_OUT: IC7.15, R18.2, R20.1
- new net FM_CLKIN: C4.2, IC7.8, Q2.2
- new net FM_CLKOUT: C5.2, IC7.9, Q2.1
- new net FM_WR: IC2B.Y3, IC7.11
- new net N$3: D1.C, IC8.1, R2.2
- new net OUT: C6.-, R4.2
- new net PSG1_LED: IC1.PD3(INT1), LED1.A
- new net PSG2_LED: IC1.PD4(XCK/T0), LED2.A
- new net PSG3_LED: IC1.PD5(T1), LED3.A
- new net PSG_CLK: IC4.7, IC5.7, IC6.7, QG1.OUT
- new net RCK: IC1.PB2(SS/OC1B), IC3A.RCK
- new net WR_A: IC1.PC2(ADC2), IC2B.A
- new net WR_B: IC1.PC3(ADC3), IC2B.B
- new net WR_E: IC1.PB1(OC1A), IC2B.G
- net A0: now also IC1.PC5(ADC5/SCL), IC6.3, IC7.10; no longer IC1.(SS)PB4, IC3.3, IC6.10
- net DATA0: now also IC3A.QA, IC6.18, IC7.17; no longer IC1.(ADC0)PA0, IC3.18, IC6.17
- net DATA1: now also IC3A.QB, IC6.17, IC7.18; no longer IC1.(ADC1)PA1, IC3.17, IC6.18
- net DATA2: now also IC3A.QC, IC6.16, IC7.2; no longer IC1.(ADC2)PA2, IC3.16, IC6.2
- net DATA3: now also IC3A.QD, IC6.15, IC7.3; no longer IC1.(ADC3)PA3, IC3.15, IC6.3
- net DATA4: now also IC3A.QE, IC6.14, IC7.4; no longer IC1.(ADC4)PA4, IC3.14, IC6.4
- net DATA5: now also IC3A.QF, IC6.13, IC7.5; no longer IC1.(ADC5)PA5, IC3.13, IC6.5
- net DATA6: now also IC3A.QG, IC6.12, IC7.6; no longer IC1.(ADC6)PA6, IC3.12, IC6.6
- net DATA7: now also IC3A.QH, IC6.11, IC7.7; no longer IC1.(ADC7)PA7, IC3.11, IC6.7
- net FM_CS: now also IC2A.Y3, IC7.12; no longer IC1.(TOSC2)PC7, IC6.12
- net GND: now also C1.1, C14.2, C2.1, C22.2, C4.1, C5.1, C7.2, IC3A.G, IC6.6, IC6.8, IC7.1, LED2.C, LED3.C, LED4.C, LED5.C, R19.2, R20.2, R7.1, R9.1, SV1.6, SV3.1, SV3.3; no longer C1.2, C2.2, C3.2, C4.2, C5.2, C6.-, C7.-, IC10.14, IC3.6, IC3.8, IC6.1, IC7.5, IC8.4, IC9.2, QG2.GND, R17.1, R19.1, R22.1, R23.1, R28.1, R29.1, SV3.2, SV4.1, SV4.3, SV5.2, SV6.6, SV7.5, T2.C, VR4.E
- net IC: now also IC1.PC4(ADC4/SDA), IC6.9, IC7.13; no longer D2.C, IC1.(AIN1/OC0)PB3, IC3.9, IC6.13
- net MIDI_IN: now also IC1.PD0(RXD), IC8.7, LED6.C; no longer IC11.8, IC7.7, LED2.C
- net MISO: now also IC1.PB4(MISO), SV1.1; no longer IC1.(MISO)PB6, SV6.1
- net MOSI: now also IC1.PB3(MOSI/OC2), IC3A.SER, SV1.4; no longer IC1.(MOSI)PB5, SV6.4
- net N$1: now also C1.2, IC1.PB6(XTAL1/TOSC1), Q1.2; no longer R2.1, SV1.4
- net N$10: now also C8.-, R8.1; no longer C10.+, C11.+, C12.+, C8.+, C9.+, IC8.2, VR3.A, VR3.S
- net N$11: now also IC4.10; no longer C5.1, R7.1, VR2.A, VR2.S
- net N$13: now also IC6.10; no longer R8.2, R9.1, T1.B
- net N$14: now also C2.2, IC1.PB7(XTAL2/TOSC2), Q1.1; no longer C7.+, D3.C, T1.E
- net N$15: now also C9.-; no longer T1.C
- net N$17: now also C10.-, R12.1; no longer C14.-, IC9.3, R23.2, T2.E
- net N$18: now also R13.2, R14.2, VR2.1; no longer R11.2, R12.2, VR2.E
- net N$19: now also C11.-, R14.1; no longer C8.-, R12.1
- net N$2: now also R2.1, SV2.4; no longer D1.A, IC7.2, SV1.5
- net N$20: now also R15.2, R16.2, VR3.1; no longer R13.2, R14.2, VR1.E
- net N$21: now also C12.-, R16.1; no longer C9.-, R14.1
- net N$22: now also C14.1, R18.1, VR3.2, VR3.3; no longer LED4.A, R25.1
- net N$23: now also C10.+, C11.+, C12.+, C8.+, C9.+, IC9.2, SV5.1; no longer C10.-, R16.1
- net N$24: now also C13.1, R17.1, VR2.2, VR2.3; no longer LED5.A, R30.1
- net N$4: now also D1.A, IC8.2, SV2.5; no longer C2.1, IC1.XTAL1, Q1.1
- net N$5: now also C3.2, IC8.5; no longer D1.C, IC7.1, R2.2
- net N$7: now also IC9.1, SV5.2, SV5.3; no longer D2.A, R8.1
- net N$8: now also IC5.10; no longer C4.1, R5.1, VR1.A, VR1.S
- net PSG1_CS: now also IC2A.Y0, IC4.2; no longer IC1.(SDA)PC1, IC3.2
- net PSG1_OUT: now also IC4.5, R7.2, R8.2; no longer IC3.5, R19.2, R20.2
- net PSG1_WR: now also IC2B.Y0, IC4.1; no longer IC1.(SCL)PC0, IC3.1
- net PSG2_CS: now also IC2A.Y1, IC5.2; no longer IC1.(TMS)PC3, IC4.2
- net PSG2_OUT: now also IC5.5, R10.2, R9.2; no longer IC4.5, R17.2, R18.2
- net PSG2_WR: now also IC2B.Y1, IC5.1; no longer IC1.(TCK)PC2, IC4.1
- net PSG3_CS: now also IC2A.Y2, IC6.2; no longer IC1.(TDI)PC5, IC5.2
- net PSG3_OUT: now also IC6.5, R11.2, R12.2; no longer IC5.5, R15.2, R16.2
- net PSG3_WR: now also IC2B.Y2, IC6.1; no longer IC1.(TDO)PC4, IC5.1
- net RST: now also IC1.PC6(/RESET), R1.2, SV1.5; no longer IC1.RESET, R1.1, SV6.5
- net SCK: now also IC1.PB5(SCK), IC3A.SCK, SV1.3; no longer IC1.(SCK)PB7, SV6.3
- net VBIAS: now also C7.1, IC9.3, R5.1, R6.2; no longer C13.1, IC8.3, R21.1, R22.2
- net VCC: now also C22.1, IC1.VCC@1, IC3A.SCL, IC6.4, IC7.16, IC9.8, LED6.A, R1.1, R5.2, SV1.2, SV3.2; no longer D3.A, IC1.VCC, IC11.5, IC11.6, IC3.4, IC6.16, IC7.8, IC9.7, QG2.VCC, R1.2, R21.2, R24.2, R25.2, R26.2, R27.2, R30.2, R9.2, SV4.2, SV5.1, SV6.2
Other:
- note added: "HiT0M1 Ver2.60"
- note removed: "0.015u capacitors use film capacitor"
- note removed: "HARDWARE MIDI TONE GENERATOR -HiT0M1"
- note removed: "Vcc=5v GND=0v"
- note removed: "Ver2.40"
- moved on the sheet: C1, C10, C11, C12, C13, C15, C16, C17, C18, C19, C2, C20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
