File: Schematic/BOARD.sch (EAGLE design)
At the start: 69 parts, among them IC1 MEGA328P, IC2 74HC139N, IC3 74HC595N, IC4 YMZ294, IC5 YMZ294, IC6 YMZ294, IC7 YM2413, IC8 TLP2630, IC9 NJM2114, Q1 16MHz, Q2 3.579545MHz

Commit message: Whole Changes
Update Readme.md and Added gerber files,change pictures of the circuit
Parts:
- removed LED2, LED3, LED4, LED5, LED6: WITH_R, led:LED3MM
- removed Q1: 16MHz, crystal:CRYSTALHC49S
- removed Q2: 3.579545MHz, crystal:CRYSTALHC49S
- removed R1: 10k, rcl:R-EU_0207/10
- added C24, C25: 10u, rcl:CPOL-EUE2,5-6E
- added IC10: NJM2114DD, ic-package:DIL8S
- added IC11: 74HC595N, 74xx-eu:74HC595N
- added QG2: 8MHz, crystal:XO-14
- added R21, R23, R25, R27, R28, R29, R31, R33, R35: 10k, rcl:R-EU_0207/2V
- added R22, R24, R26, R30, R32, R34: 1.2k, rcl:R-EU_0207/2V
- added VR1: P-03277_VR_3362P, Akizuki:P-03277_VR_3362P
- added VR4, VR5, VR6, VR7, VR8: VR_3362P, Akizuki:P-03277_VR_3362P
- C1, C2, C4, C5: value 22p -> 0.1u
- C10, C8, C9: value 10u -> 0.015u; device rcl:CPOL-EUE2.5-6 -> rcl:C-EU050-025X075
- C11, C12: value 10u -> 0.1u; device rcl:CPOL-EUE2.5-6 -> rcl:C-EU025-025X050
- C13: value 0.015u -> 10u; device rcl:C-EU050-025X075 -> rcl:CPOL-EUE2,5-6E
- C15, C16: value 0.1u -> 0.015u; device rcl:C-EU025-025X050 -> rcl:C-EU050-025X075
- C17, C22: value 0.1u -> 100u; device rcl:C-EU025-025X050 -> rcl:CPOL-EUE2,5-6E
- C18, C19, C20, C7: value 0.1u -> 10u; device rcl:C-EU025-025X050 -> rcl:CPOL-EUE2,5-6E
- C23: value 470u -> 10u; device rcl:CPOL-EUE2.5-6 -> rcl:CPOL-EUE2,5-6E
- C6: value 100u -> 0.1u; device rcl:CPOL-EUE2.5-6 -> rcl:C-EU025-025X050
- IC1: value MEGA328P -> YM2413; device atmel:MEGA8-P -> ic-package:DIL18S
- IC2: value 74HC139N -> F303K8; device 74xx-eu:74HC139N -> ic-package:DIL32
- IC3: value 74HC595N -> YM2413; device 74xx-eu:74HC595N -> ic-package:DIL18S
- IC4: value YMZ294 -> YM2413
- IC5: value YMZ294 -> AE-LLCNV8; device ic-package:DIL18S -> ic-package:DIL20S
- IC7: value YM2413 -> TLP2630; device ic-package:DIL18S -> ic-package:DIL8S
- IC8: value TLP2630 -> YMZ294; device ic-package:DIL8S -> ic-package:DIL18S
- IC9: value NJM2114 -> AE-LLCNV8; device ic-package:DIL8S -> ic-package:DIL20S
- LED1: value WITH_R -> WITHR
- QG1: value 8MHz -> 3.579545MHz
- R11, R13: value 1.2k -> 4.7k
- R12: value 10k -> 2.2k
- R14, R16: value 10k -> 4.7k
- R15: value 1.2k -> 2.2k
- R17: value 4.7k -> 2.2k
- R2: value 220 -> 1.2k; device rcl:R-EU_0207/10 -> rcl:R-EU_0207/2V
- R20: value 2.2k -> 10k
- R3: value 1k -> 2.2k; device rcl:R-EU_0207/10 -> rcl:R-EU_0207/2V
- R4: value 10k -> 2.2k; device rcl:R-EU_0207/10 -> rcl:R-EU_0207/2V
- R5: value 10k -> 4.7k; device rcl:R-EU_0207/10 -> rcl:R-EU_0207/2V
- R6: value 10k -> 220; device rcl:R-EU_0207/10 -> rcl:R-EU_0207/2V
- R7: value 1.2k -> 1k
- SV1: value ICSP -> MIDI; device con-lstb:MA03-2 -> con-lstb:MA05-1
- SV2: value MIDI_IN -> 3V3C; device con-lstb:MA05-1 -> con-lstb:MA03-1
- SV3: value POWER -> 5vIN
- SV4: value OUT -> VOL
- SV5: value VOL -> OUT
Connections:
- removed net CS_A: IC1.PC0(ADC0), IC2A.A
- removed net CS_B: IC1.PC1(ADC1), IC2A.B
- removed net CS_E: IC1.PB0(ICP), IC2A.G
- removed net DATA0: IC3A.QA, IC4.18, IC5.18, IC6.18, IC7.17
- removed net DATA1: IC3A.QB, IC4.17, IC5.17, IC6.17, IC7.18
- removed net DATA2: IC3A.QC, IC4.16, IC5.16, IC6.16, IC7.2
- removed net DATA3: IC3A.QD, IC4.15, IC5.15, IC6.15, IC7.3
- removed net DATA4: IC3A.QE, IC4.14, IC5.14, IC6.14, IC7.4
- removed net DATA5: IC3A.QF, IC4.13, IC5.13, IC6.13, IC7.5
- removed net DATA6: IC3A.QG, IC4.12, IC5.12, IC6.12, IC7.6
- removed net DATA7: IC3A.QH, IC4.11, IC5.11, IC6.11, IC7.7
- removed net FMM_LED: IC1.PD7(AIN1), LED5.A
- removed net FMM_OUT: IC7.14, R17.2, R19.1
- removed net FMR_LED: IC1.PD6(AIN0), LED4.A
- removed net FMR_OUT: IC7.15, R18.2, R20.1
- removed net FM_CLKIN: C4.2, IC7.8, Q2.2
- removed net FM_CLKOUT: C5.2, IC7.9, Q2.1
- removed net FM_CS: IC2A.Y3, IC7.12
- removed net FM_WR: IC2B.Y3, IC7.11
- removed net MIDI_IN: IC1.PD0(RXD), IC8.7, LED6.C, R3.1
- removed net MISO: IC1.PB4(MISO), SV1.1
- removed net MOSI: IC1.PB3(MOSI/OC2), IC3A.SER, SV1.4
- removed net N$3 (its old number): D1.C, IC8.1, R2.2
- removed net PSG1_CS: IC2A.Y0, IC4.2
- removed net PSG1_LED: IC1.PD3(INT1), LED1.A
- removed net PSG1_WR: IC2B.Y0, IC4.1
- removed net PSG2_CS: IC2A.Y1, IC5.2
- removed net PSG2_LED: IC1.PD4(XCK/T0), LED2.A
- removed net PSG2_WR: IC2B.Y1, IC5.1
- removed net PSG3_CS: IC2A.Y2, IC6.2
- removed net PSG3_LED: IC1.PD5(T1), LED3.A
- removed net PSG3_OUT: IC6.5, R11.2, R12.2
- removed net PSG3_WR: IC2B.Y2, IC6.1
- removed net RCK: IC1.PB2(SS/OC1B), IC3A.RCK
- removed net RST: IC1.PC6(/RESET), R1.2, SV1.5
- removed net WR_A: IC1.PC2(ADC2), IC2B.A
- removed net WR_B: IC1.PC3(ADC3), IC2B.B
- removed net WR_E: IC1.PB1(OC1A), IC2B.G
- new net +5V: C11.1, C2.1, C3.1, C4.1, C6.1, IC1.16, IC10.8, IC3.16, IC4.16, IC5.20, IC6.4, IC8.4, IC9.20, QG1.VCC, QG2.VCC, R29.2, SV2.1, SV3.2
- new net 3V3_A0: IC2.12, IC5.8
- new net 3V3_IC: IC2.11, IC5.7
- new net 3V3_WRCS_FM1: IC2.8, IC5.4
- new net 3V3_WRCS_FM2: IC2.9, IC5.5
- new net 3V3_WRCS_FM3: IC2.10, IC5.6
- new net 3V3_WRCS_PSG1: IC2.6, IC5.2
- new net 3V3_WRCS_PSG2: IC2.7, IC5.3
- new net D0: IC1.17, IC3.17, IC4.17, IC6.18, IC8.18, IC9.19
- new net D1: IC1.18, IC3.18, IC4.18, IC6.17, IC8.17, IC9.18
- new net D2: IC1.2, IC3.2, IC4.2, IC6.16, IC8.16, IC9.17
- new net D3: IC1.3, IC3.3, IC4.3, IC6.15, IC8.15, IC9.16
- new net D4: IC1.4, IC3.4, IC4.4, IC6.14, IC8.14, IC9.15
- new net D5: IC1.5, IC3.5, IC4.5, IC6.13, IC8.13, IC9.14
- new net D6: IC1.6, IC3.6, IC4.6, IC6.12, IC8.12, IC9.13
- new net D7: IC1.7, IC3.7, IC4.7, IC6.11, IC8.11, IC9.12
- new net FM1_MOUT: IC4.14, R17.2, R5.1
- new net FM1_ROUT: IC4.15, R18.1, R19.2
- new net FM1_WRCS: IC4.11, IC4.12, IC5.17
- new net FM2_MOUT: IC3.14, R14.1, R4.2
- new net FM2_ROUT: IC3.15, R15.2, R16.1
- new net FM2_WRCS: IC3.11, IC3.12, IC5.16
- new net FM3_MOUT: IC1.14, R11.1, R3.2
- new net FM3_ROUT: IC1.15, R12.2, R13.1
- new net FM3_WRCS: IC1.11, IC1.12, IC5.15
- new net FM_CLK: IC1.8, IC3.8, IC4.8, QG1.OUT
- new net N$12: IC11A.QD, IC9.5
- new net N$13: IC11A.QE, IC9.6
- new net N$16: IC11A.QH, IC9.9
- new net N$25: C20.-, R27.1
- new net N$26: C25.-, R35.2
- new net N$27: IC4.9
- new net N$28: C19.-, R25.1
- new net N$29: C24.-, R33.2
- new net N$30: C19.+, C20.+, C24.+, C25.+, IC10.2, VR5.2, VR5.3
- new net N$31: C8.1, R11.2, VR6.1, VR6.2
- new net N$33: R22.1, R23.1, VR6.3
- new net N$34: C18.-, R23.2
- new net N$35: C14.1, R13.2, VR2.1, VR2.2
- new net N$37: R30.1, R31.1, VR2.3
- new net N$38: C23.-, R31.2
- new net N$40: C7.-, R8.2
- new net N$42: C13.-, R10.2
- new net N$45: SV4.3, SV5.1, SV5.3
- new net N$48: C17.+, IC10.1, VR5.1
- new net N$49: C22.+, IC10.7, VR1.3
- new net N$6: IC3.9
- new net N$9: IC11A.QC, IC9.4
- new net PSG1_WRCS: IC5.19, IC8.1, IC8.2
- new net PSG2_WRCS: IC5.18, IC6.1, IC6.2
- new net RCLK: IC11A.RCK, IC2.5
- new net RXD: IC2.2, IC7.7, LED1.C, R7.2
- new net SER: IC11A.SER, IC2.15
- net A0: now also IC1.10, IC3.10, IC4.10, IC5.13, IC8.3; no longer IC1.PC5(ADC5/SCL), IC4.3, IC5.3, IC7.10
- net GND: now also C1.2, C10.2, C11.2, C12.2, C2.2, C3.2, C4.2, C5.2, C6.2, C8.2, C9.2, IC1.1, IC10.4, IC11A.G, IC2.31, IC2.4, IC3.1, IC4.1, IC5.10, IC5.11, IC7.5, IC8.6, IC8.8, IC9.10, IC9.11, QG2.GND, R12.1, R17.1, R19.1, R2.2, R20.1, R21.1, R22.2, R24.1, R26.1, R28.1, R3.1, R30.2, R32.2, R34.2, R9.2, SV2.2, SV4.1, SV5.2; no longer C1.1, C13.2, C17.2, C18.2, C19.2, C2.1, C20.2, C22.2, C23.-, C4.1, C5.1, C7.2, IC1.AREF, IC1.GND, IC1.GND@1, IC3A.G, IC4.6, IC4.8, IC5.6, IC5.8, IC7.1, IC9.4, LED1.C, LED2.C, LED3.C, LED4.C, LED5.C, R11.1, R13.1, R19.2, R20.2, R6.1, R7.1, R9.1, SV1.6
- net IC: now also IC1.13, IC3.13, IC4.13, IC5.14, IC8.9; no longer IC1.PC4(ADC4/SDA), IC4.9, IC5.9, IC7.13
- net N$1: now also C10.1, R5.2, VR8.1, VR8.2; no longer C1.2, IC1.PB6(XTAL1/TOSC1), Q1.2
- net N$10: now also IC8.10; no longer C8.-, R8.1
- net N$11: now also IC1.9; no longer IC4.10
- net N$14: now also IC11A.QF, IC9.7; no longer C2.2, IC1.PB7(XTAL2/TOSC2), Q1.1
- net N$15: now also IC11A.QG, IC9.8; no longer C9.-, R10.1
- net N$17: now also C9.1, R14.2, VR7.1, VR7.2; no longer C10.-, R12.1
- net N$18: now also D1.A, IC7.2, SV1.5; no longer R13.2, R14.2, VR2.1
- net N$19: now also C15.1, R16.2, VR3.1, VR3.2; no longer C11.-, R14.1
- net N$2: now also D1.C, IC7.1, R6.2; no longer R2.1, SV2.4
- net N$20: now also C13.+, C18.+, C23.+, C7.+, IC10.6, VR1.1, VR1.2; no longer R15.2, R16.2, VR3.1
- net N$21: now also R32.1, R33.1, VR3.3; no longer C12.-, R16.1
- net N$22: now also R24.2, R25.2, VR7.3; no longer C14.1, R18.1, VR3.2, VR3.3
- net N$23: now also R34.1, R35.1, VR4.3; no longer C10.+, C11.+, C12.+, C8.+, C9.+, IC9.2, SV5.1
- net N$24: now also R26.2, R27.2, VR8.3; no longer C13.1, R17.1, VR2.2, VR2.3
- net N$4: now also C16.1, R18.2, VR4.1, VR4.2; no longer D1.A, IC8.2, SV2.5
- net N$5: now also R6.1, SV1.4; no longer C3.2, IC8.5
- net N$7: now also IC11A.QA, IC9.2; no longer C6.+, IC9.1, SV5.2, SV5.3
- net N$8: now also IC11A.QB, IC9.3; no longer IC5.10
- net OUT: now also C17.-, C22.-, R20.2, R21.2, SV4.2; no longer C6.-, R4.2
- net PSG1_OUT: now also IC8.5, R2.1, R8.1; no longer IC4.5, R7.2, R8.2
- net PSG2_OUT: now also IC6.5, R10.1, R9.1; no longer IC5.5, R10.2, R9.2
- net PSG_CLK: now also IC8.7, QG2.OUT; no longer IC4.7, IC5.7, QG1.OUT
- net SCK: now also IC11A.SCK, IC2.18; no longer IC1.PB5(SCK), IC3A.SCK, SV1.3
- net VBIAS: now also C12.1, IC10.3, IC10.5, R28.2, R29.1; no longer C7.1, IC9.3, R5.1, R6.2
- net VCC: now also C1.1, C5.1, IC11A.SCL, IC2.19, IC5.1, IC7.8, IC9.1, LED1.A, R7.1, SV2.3; no longer C15.1, C16.1, C17.1, C18.1, C19.1, C20.1, C22.1, C23.+, C3.1, IC1.AVCC, IC1.VCC@1, IC3A.SCL, IC4.4, IC5.4, IC6.4, IC7.16, IC8.8, IC9.8, LED6.A, QG1.VCC, R1.1, R3.2, R5.2, SV1.2, SV3.2
Other:
- note added: "3.29"
- note added: "F"
- note added: "HiT0M1-Fast"
- note added: "VCC=3.3V"
- note removed: "HiT0M1 Ver2.60"
- moved on the sheet: C1, C14, C15, C16, C2, C21, C23, C3, C4, C5, D1, IC4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
